File: ESP31.kicad_sch (KiCad schematic)
At the start: 48 parts, among them J25 Conn_01x01, J26 Conn_01x01, J27 Conn_01x01, J28 Conn_01x01, J29 Conn_01x01, J30 Conn_01x01, J31 Conn_01x01, J32 Conn_01x01, J33 Conn_01x01, J34 Conn_01x01, J35 Conn_01x01, J36 Conn_01x01, J40 Conn_01x01, J41 Conn_01x01, J42 Conn_01x01, J43 Conn_01x01, J44 Conn_01x01, J45 Conn_01x01, J46 Conn_01x01, J47 Conn_01x01, J48 Conn_01x01, J49 Conn_01x01, J50 Conn_01x01, J51 Conn_01x01, J52 Conn_01x01, J53 Conn_01x01, J54 Conn_01x01, J55 Conn_01x01, J56 Conn_01x01, J57 Conn_01x01, J58 Conn_01x01, J59 Conn_01x01, J60 Conn_01x01, J61 Conn_01x01, J62 Conn_01x01, J63 Conn_01x01, SW1 SW_Push, SW2 SW_Push, U1 ESP32-PICO-D4

Commit message: Final Version
Last ordered version. It's working :)
Parts:
- removed C4, C5: 100n, Capacitor_SMD:C_0603_1608Metric, symbol Device:C
- removed J25, J26, J27, J28, J29, J30, J31, J32, J33, J34, J35, J36, J40, J41, J42, J43, J44, J45, J46, J47, J48, J49, J50, J51, J52, J53, J54, J55, J56, J57, J58, J59, J60, J61, J62, J63, J?: Conn_01x01, Connector_PinHeader_1.00mm:PinHeader_1x01_P1.00mm_Vertical, symbol Connector_Generic:Conn_01x01
- removed R2: 10K, Resistor_SMD:R_0603_1608Metric, symbol Device:R
- added D1: WS2812B_Geaendertes_Symbol, LED_SMD:LED_Cree-PLCC4_2x2mm_CW, symbol TheBrutzlers_Lib:WS2812B_Geaendertes_Symbol
- added J1: Conn_02x04_Odd_Even, Connector_PinHeader_2.54mm:PinHeader_2x04_P2.54mm_Vertical, symbol Connector_Generic:Conn_02x04_Odd_Even
- added J10, J11, J12, J13, J14, J15, J16, J17, J18, J19, J20, J21, J22, J23, J24, J3, J4, J5, J6: Conn_01x01, Eigene:CON_1x01, symbol Connector_Generic:Conn_01x01
- C1, C3: LCSC (none) -> C282519
- C2: LCSC (none) -> C85713
- R1: LCSC (none) -> C73809
- SW1, SW2: footprint Button_Switch_SMD:SW_DIP_SPSTx01_Slide_6.7x4.1mm_W8.61mm_P2.54mm_LowProfile -> TheBrutzlers_Lib:microswitch; LCSC (none) -> C100056
Connections:
- net +3V3: now also D1.4 (VDD), J1.8 (Pin_8)
- net CAPN: now also J5.1 (Pin_1)
- net CAPP: now also J4.1 (Pin_1)
- net EN: now also J1.6 (Pin_6)
- net GND: now also D1.2 (VSS), J1.1 (Pin_1)
- net IO0: now also J1.5 (Pin_5)
- net IO1: now also J1.2 (Pin_2)
- net IO10: now also J12.1 (Pin_1)
- net IO18: now also J13.1 (Pin_1)
- net IO19: now also J14.1 (Pin_1)
- net IO2: now also D1.3 (DIN), J1.3 (Pin_3)
- net IO21: now also J15.1 (Pin_1)
- net IO22: now also J16.1 (Pin_1)
- net IO23: now also J17.1 (Pin_1)
- net IO25: now also J18.1 (Pin_1)
- net IO26: now also J19.1 (Pin_1)
- net IO27: now also J20.1 (Pin_1)
- net IO3: now also J1.7 (Pin_7)
- net IO32: now also J21.1 (Pin_1)
- net IO33: now also J22.1 (Pin_1)
- net IO34: now also J23.1 (Pin_1)
- net IO35: now also J24.1 (Pin_1)
- net IO4: now also J1.4 (Pin_4)
- net IO5: now also J10.1 (Pin_1)
- net IO9: now also J11.1 (Pin_1)
- net SENS_VN: now also J6.1 (Pin_1)
- net SENS_VP: now also J3.1 (Pin_1)
- net CMD: no longer names the net of U1.30 (CMD)
- net IO17: no longer names the net of U1.27 (IO17)
- net MTCK: no longer names the net of U1.20 (IO13)
- net MTDI: no longer names the net of U1.18 (IO12)
- net MTDO: no longer names the net of U1.21 (IO15)
- net MTMS: no longer names the net of U1.17 (IO14)
- net SD0: no longer names the net of U1.32 (SD0)
- net SD1: no longer names the net of U1.33 (SD1)
- no-connect marks 1 -> 0
Other:
- note removed: "BOOTMODE"
- note removed: "RESET"
- moved on the sheet: C2, C3
