File: ESP31_V3.kicad_pcb (KiCad board)
At the start: 4 copper layers, 20 x 25 mm, 49 parts, among them J1 Conn_01x01, J10 Conn_01x01, J11 Conn_01x01, J12 Conn_01x01, J13 Conn_01x01, J14 Conn_01x01, J15 Conn_01x01, J16 Conn_01x01, J17 Conn_01x01, J18 Conn_01x01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

Commit message: corrected WS2812 Footprint
corrected WS2812 Footprint
switched input and output of RGB LED
Connections:
- D1 pad 1: /IO2 -> unconnected-(D1-Pad1)
- D1 pad 3: unconnected-(D1-Pad3) -> /IO2
Routing:
- net /IO2: track 28.2 -> 25.2 mm
Changed lines of the file:
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@@
   (net 9 "/IO3")
   (net 10 "Net-(C1-Pad2)")
-  (net 11 "unconnected-(D1-Pad3)")
+  (net 11 "unconnected-(D1-Pad1)")
   (net 12 "unconnected-(U2-Pad48)")
   (net 13 "unconnected-(U2-Pad47)")
@@
     (descr "QFN, 48 Pin (https://www.trinamic.com/fileadmin/assets/Products/ICs_Documents/TMC2041_datasheet.pdf#page=62), generated with kicad-footprint-generator ipc_noLead_generator.py")
     (tags "QFN NoLead")
+    (property "LCSC" " C193707 ")
     (property "Sheetfile" "ESP31_V3.kicad_sch")
     (property "Sheetname" "")
@@
   (footprint "TheBrutzlers_Lib:microswitch" (layer "F.Cu")
     (at 117.856 113.284 -90)
-    (property "LCSC" "C100056")
+    (property "LCSC" "C482003")
     (property "Sheetfile" "ESP31_V3.kicad_sch")
     (property "Sheetname" "")
@@
     (fp_circle (center 0 0) (end 0.8 0) (layer "F.Fab") (width 0.1) (fill none))
     (pad "1" smd rect locked (at -0.75 -0.55 270) (size 1 0.8) (layers "F.Cu" "F.Paste" "F.Mask")
-      (net 6 "/IO2") (pinfunction "DI") (pintype "input"))
+      (net 11 "unconnected-(D1-Pad1)") (pinfunction "DOUT") (pintype "output"))
     (pad "2" smd rect locked (at -0.75 0.55 270) (size 1 0.8) (layers "F.Cu" "F.Paste" "F.Mask")
       (net 1 "GND") (pinfunction "VSS") (pintype "power_in"))
     (pad "3" smd rect locked (at 0.75 0.55 270) (size 1 0.8) (layers "F.Cu" "F.Paste" "F.Mask")
-      (net 11 "unconnected-(D1-Pad3)") (pinfunction "DO") (pintype "output"))
+      (net 6 "/IO2") (pinfunction "DIN") (pintype "input"))
     (pad "4" smd rect locked (at 0.75 -0.55 270) (size 1 0.8) (layers "F.Cu" "F.Paste" "F.Mask")
       (net 4 "+3V3") (pinfunction "VDD") (pintype "power_in"))
@@
     (fp_line (start 2.3 -1.25) (end 2.3 1.25) (layer "B.CrtYd") (width 0.05))
     (pad "1" smd custom locked (at -1.3 0 270) (size 1 0.5) (layers "B.Cu" "B.Mask")
-      (net 4 "+3V3") (pinfunction "A") (zone_connect 2)
+      (net 4 "+3V3") (pinfunction "A") (pintype "passive") (zone_connect 2)
       (options (clearance outline) (anchor rect))
       (primitives
@@
       ))
     (pad "2" smd rect locked (at 0 0 270) (size 1 1.5) (layers "B.Cu" "B.Mask")
-      (net 46 "VIN") (pinfunction "C"))
+      (net 46 "VIN") (pinfunction "C") (pintype "input"))
     (pad "3" smd custom locked (at 1.3 0 270) (size 1 0.5) (layers "B.Cu" "B.Mask")
-      (net 10 "Net-(C1-Pad2)") (pinfunction "B") (zone_connect 2)
+      (net 10 "Net-(C1-Pad2)") (pinfunction "B") (pintype "passive") (zone_connect 2)
       (options (clearance outline) (anchor rect))
       (primitives
@@
   (segment (start 114.099511 110.044213) (end 114.849832 109.293892) (width 0.2) (layer "B.Cu") (net 5))
   (segment (start 113.6 112) (end 113.970489 111.629511) (width 0.2) (layer "B.Cu") (net 5))
+  (segment (start 116.0042 99.6442) (end 115.5446 99.6442) (width 0.2) (layer "F.Cu") (net 6))
   (segment (start 107.565948 104.75) (end 108.05 104.75) (width 0.2) (layer "F.Cu") (net 6))
-  (segment (start 117.7 98.59) (end 117.7 97.7) (width 0.2) (layer "F.Cu") (net 6))
+  (segment (start 116.45 100.09) (end 116.0042 99.6442) (width 0.2) (layer "F.Cu") (net 6))
   (segment (start 106.950961 105.364987) (end 107.565948 104.75) (width 0.2) (layer "F.Cu") (net 6))
   (segment (start 106.950961 108.050961) (end 106.950961 105.364987) (width 0.2) (layer "F.Cu") (net 6))
   (segment (start 107.06974 108.16974) (end 106.950961 108.050961) (width 0.2) (layer "F.Cu") (net 6))
-  (segment (start 117.7 97.7) (end 117.8 97.6) (width 0.2) (layer "F.Cu") (net 6))
   (via (at 107.06974 108.16974) (size 0.4) (drill 0.3) (layers "F.Cu" "B.Cu") (net 6))
-  (via (at 117.8 97.6) (size 0.4) (drill 0.3) (layers "F.Cu" "B.Cu") (net 6))
-  (segment (start 108.91 105.69) (end 108.91 101.18) (width 0.2) (layer "B.Cu") (net 6))
-  (segment (start 114.52 100.88) (end 117.8 97.6) (width 0.2) (layer "B.Cu") (net 6))
+  (via (at 115.5446 99.6442) (size 0.4) (drill 0.3) (layers "F.Cu" "B.Cu") (net 6))
+  (segment (start 107.06974 107.53026) (end 108.91 105.69) (width 0.2) (layer "B.Cu") (net 6))
   (segment (start 107.06974 108.16974) (end 107.06974 107.53026) (width 0.2) (layer "B.Cu") (net 6))
-  (segment (start 109.21 100.88) (end 114.52 100.88) (width 0.2) (layer "B.Cu") (net 6))
   (segment (start 107.06974 108.16974) (end 107.4 108.5) (width 0.2) (layer "B.Cu") (net 6))
-  (segment (start 107.06974 107.53026) (end 108.91 105.69) (width 0.2) (layer "B.Cu") (net 6))
+  (segment (start 109.21 100.88) (end 114.3088 100.88) (width 0.2) (layer "B.Cu") (net 6))
+  (segment (start 114.3088 100.88) (end 115.5446 99.6442) (width 0.2) (layer "B.Cu") (net 6))
   (segment (start 110.04 109.350723) (end 110.04 110.725) (width 0.2) (layer "B.Cu") (net 6))
   (segment (start 109.189277 108.5) (end 110.04 109.350723) (width 0.2) (layer "B.Cu") (net 6))
   (segment (start 108.91 101.18) (end 109.21 100.88) (width 0.2) (layer "B.Cu") (net 6))
   (segment (start 107.4 108.5) (end 109.189277 108.5) (width 0.2) (layer "B.Cu") (net 6))
+  (segment (start 108.91 105.69) (end 108.91 101.18) (width 0.2) (layer "B.Cu") (net 6))
   (segment (start 107.968771 105.831229) (end 108.05 105.75) (width 0.2) (layer "F.Cu") (net 7))
   (segment (start 107.968771 108.716386) (end 107.968771 105.831229) (width 0.2) (layer "F.Cu") (net 7))
