File: ESP31_V3.kicad_sch (KiCad schematic)
At the start: 32 parts, among them J1 Conn_01x01, J10 Conn_01x01, J11 Conn_01x01, J12 Conn_01x01, J13 Conn_01x01, J14 Conn_01x01, J15 Conn_01x01, J16 Conn_01x01, J17 Conn_01x01, J18 Conn_01x01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

Commit message: corrected WS2812 Footprint
corrected WS2812 Footprint
switched input and output of RGB LED
Connections:
- net IO2: now also D1.3 (DIN); no longer D1.1 (DI)
